File: FEEDERLINK.brd (EAGLE design)
At the start: 54 x 15 mm, 5 parts, among them J5 M02X5-SHROUDED

Commit message: Changed net names to match functions
Connections:
- net D0 renamed FB0
- net D1 renamed SIG0
- net D2 renamed FB1
- net D3 renamed SIG1
- net D4 renamed FB2
- net D5 renamed SIG2
- net D6 renamed FB3
- net D7 renamed SIG3
Other:
- board text added: "0"
- board text removed: "4"
Changed lines of the file:
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@@
 </layers>
 <board>
-<fusionsync huburn="a.cGVyc29uYWw6dWUyZDliZmNi" projecturn="a.cGVyc29uYWw6dWUyZDliZmNiIzIwMTgwOTI2MTUwOTQ2NTA2" f3durn="urn:adsk.wipprod:dm.lineage:QDbJOjaCQIiw4yWXuLCKeQ" pcbguid="374eda25-35df-4a59-99bf-fb84bf2e6657" lastpulledtime="" lastsyncedchangeguid="9ba0060d-c17b-e3b2-e533-83580c7e3127"/>
+<fusionsync huburn="a.cGVyc29uYWw6dWUyZDliZmNi" projecturn="a.cGVyc29uYWw6dWUyZDliZmNiIzIwMTgwOTI2MTUwOTQ2NTA2" f3durn="urn:adsk.wipprod:dm.lineage:QDbJOjaCQIiw4yWXuLCKeQ" pcbguid="374eda25-35df-4a59-99bf-fb84bf2e6657" lastpulledtime="" lastsyncedchangeguid="e12e62dd-e39d-5aaa-7541-f88833778ceb"/>
 <plain>
 <wire x1="0" y1="3" x2="3" y2="0" width="0" layer="20" curve="90"/>
@@
 <wire x1="39.94" y1="7.742" x2="40.702" y2="7.996" width="0.3048" layer="21"/>
 <wire x1="40.702" y1="7.996" x2="41.21" y2="7.996" width="0.3048" layer="21"/>
-<text x="5.286" y="8.366" size="1.6764" layer="21" font="vector" ratio="18" rot="SR0">1</text>
-<text x="19.286" y="8.366" size="1.6764" layer="21" font="vector" ratio="18" rot="SR0">2</text>
-<text x="33.286" y="8.366" size="1.6764" layer="21" font="vector" ratio="18" rot="SR0">3</text>
-<text x="47.286" y="8.366" size="1.6764" layer="21" font="vector" ratio="18" rot="SR0">4</text>
+<text x="5.286" y="8.366" size="1.6764" layer="21" font="vector" ratio="18" rot="SR0">0</text>
+<text x="19.286" y="8.366" size="1.6764" layer="21" font="vector" ratio="18" rot="SR0">1</text>
+<text x="33.286" y="8.366" size="1.6764" layer="21" font="vector" ratio="18" rot="SR0">2</text>
+<text x="47.286" y="8.366" size="1.6764" layer="21" font="vector" ratio="18" rot="SR0">3</text>
 </plain>
 <attributes>
@@
 <contactref element="J5" pad="10"/>
 </signal>
-<signal name="D0">
+<signal name="FB0">
 <contactref element="J5" pad="1"/>
 <contactref element="J1" pad="4"/>
@@
 <wire x1="21.92" y1="7.27" x2="14.35" y2="7.27" width="0.4064" layer="16"/>
 </signal>
-<signal name="D1">
+<signal name="SIG0">
 <contactref element="J5" pad="2"/>
 <contactref element="J1" pad="3"/>
@@
 <wire x1="21.92" y1="4.73" x2="14.35" y2="4.73" width="0.4064" layer="16"/>
 </signal>
-<signal name="D2">
+<signal name="FB1">
 <contactref element="J5" pad="3"/>
 <contactref element="J2" pad="4"/>
@@
 <wire x1="24.46" y1="11.16" x2="23.62" y2="12" width="0.4064" layer="16"/>
 </signal>
-<signal name="D4">
+<signal name="FB2">
 <contactref element="J5" pad="5"/>
 <contactref element="J3" pad="4"/>
@@
 <wire x1="35.62" y1="10" x2="29.73" y2="10" width="0.4064" layer="1"/>
 </signal>
-<signal name="D6">
+<signal name="FB3">
 <contactref element="J5" pad="7"/>
 <contactref element="J4" pad="4"/>
@@
 <wire x1="39" y1="10" x2="49.62" y2="10" width="0.4064" layer="1"/>
 </signal>
-<signal name="D3">
+<signal name="SIG1">
 <contactref element="J5" pad="4"/>
 <contactref element="J2" pad="3"/>
@@
 <wire x1="20" y1="10.92" x2="21.08" y2="12" width="0.4064" layer="1"/>
 </signal>
-<signal name="D5">
+<signal name="SIG2">
 <contactref element="J5" pad="6"/>
 <contactref element="J3" pad="3"/>
@@
 <wire x1="25.7" y1="6.03" x2="25.7" y2="8.7" width="0.4064" layer="16"/>
 </signal>
-<signal name="D7">
+<signal name="SIG3">
 <contactref element="J5" pad="8"/>
 <contactref element="J4" pad="3"/>
